Commit message: modify urdf file and state_publisher to get closer to desired state

File: ros2_ws/src/urdf_lunabot/urdf/robot.urdf (robot description, URDF)
Before this commit: robot prototype, 1 links, 0 joints
Links:
- link base_link: geometry visual mesh filename=file://$(find urdf_lunabot)/meshes/prototype_drivetrain.stl scale=0.001 0.001 0.001
