Commit message: update luna_urdf package to include sdf, and update robot

File: ros2_ws/src/luna_urdf/luna_urdf/robot.urdf (robot description, URDF)
Before this commit: robot luna_urdf, 10 links, 9 joints
Links:
- link body: mass 25 -> 25.000000000000007105
- link wheelpod: mass 0.49999999999999983347 -> 0.5
- link wheelpod_2: mass 0.49999999999999983347 -> 0.5
- link wheelpod_3: mass 0.49999999999999983347 -> 0.5
- link wheelpod_4: mass 0.49999999999999983347 -> 0.5
Joints:
- joint steer_bl: limit effort=1 velocity=20 -> lower=-1.6580627893946131568 upper=1.6580627893946131568 effort=1 velocity=20
- joint steer_br: limit effort=1 velocity=20 -> lower=-1.6580627893946131568 upper=1.6580627893946131568 effort=1 velocity=20
- joint steer_fl: limit effort=1 velocity=20 -> lower=-1.6580627893946131568 upper=1.6580627893946131568 effort=1 velocity=20
- joint steer_fr: limit effort=1 velocity=20 -> lower=-1.6580627893946131568 upper=1.6580627893946131568 effort=1 velocity=20

Commit message: robot spawns in gazebo, controllers activated but not controlling?

File: ros2_ws/src/luna_urdf/luna_urdf/robot.urdf (robot description, URDF)
Before this commit: robot lunabot, 10 links, 9 joints
Joints:
- joint base_link_to_base: origin xyz=0 0 0 rpy=0.0 0 0 -> xyz=0 0.5 0 rpy=0.0 0 0
- joint drive_bl: limit effort=1 velocity=20 -> effort=10 velocity=20
- joint drive_br: limit effort=1 velocity=20 -> effort=10 velocity=20
- joint drive_fl: limit effort=1 velocity=20 -> effort=10 velocity=20
- joint drive_fr: limit effort=1 velocity=20 -> effort=10 velocity=20
- joint steer_bl: limit lower=-1.6580627893946131568 upper=1.6580627893946131568 effort=1 velocity=20 -> lower=-1.6580627893946131568 upper=1.6580627893946131568 effort=10 velocity=20
- joint steer_br: limit lower=-1.6580627893946131568 upper=1.6580627893946131568 effort=1 velocity=20 -> lower=-1.6580627893946131568 upper=1.6580627893946131568 effort=10 velocity=20
- joint steer_fl: limit lower=-1.6580627893946131568 upper=1.6580627893946131568 effort=1 velocity=20 -> lower=-1.6580627893946131568 upper=1.6580627893946131568 effort=10 velocity=20
- joint steer_fr: limit lower=-1.6580627893946131568 upper=1.6580627893946131568 effort=1 velocity=20 -> lower=-1.6580627893946131568 upper=1.6580627893946131568 effort=10 velocity=20
