Commit message: progress commit on lunabot_2425

File: ros2_ws/src/lunabot_2425/description/gz_control.xacro (robot description, xacro)
@@ -9,14 +9,23 @@
             <right_joint>front_right_drive_joint</right_joint>
             <wheel_separation>0.531</wheel_separation>
-            <wheel_diameter>0.2</wheel_diameter>
+            <wheel_radius>0.1</wheel_radius>
             <!-- Limits -->
-            <max_wheel_torque>20000</max_wheel_torque>
-            <max_wheel_acceleration>100</max_wheel_acceleration>
+            <max_linear_acceleration>1</max_linear_acceleration>
+            <!-- Inputs -->
+            <topic>cmd_vel</topic>
             <!-- Outputs -->
-            <odometry_frame>/odom</odometry_frame>
-            <robot_base_frame>/base_link</robot_base_frame>
-            <publish_odom>true</publish_odom>
-            <publish_odom_tf>true</publish_odom_tf>
-            <publish_wheel_tf>true</publish_wheel_tf>
+            <frame_id>odom</frame_id>
+            <child_frame_id>base_link</child_frame_id>
+            <odom_topic>odom</odom_topic>
+            <odom_publisher_frequency>30</odom_publisher_frequency>
+            <tf_topic>tf</tf_topic>
+        </plugin>
+        <plugin filename="gz-sim-joint-state-publisher-system"
+            name="gz::sim::systems::JointStatePublisher">
+            <topic>joint_states</topic>
+            <joint_name>rear_left_drive_joint</joint_name>
+            <joint_name>front_left_drive_joint</joint_name>
+            <joint_name>rear_right_drive_joint</joint_name>
+            <joint_name>front_right_drive_joint</joint_name>
         </plugin>
     </gazebo>

File: ros2_ws/src/lunabot_2425/description/robot.urdf.xacro (robot description, xacro)
@@ -2,4 +2,6 @@
 <robot xmlns:xacro="http://www.ros.org/wiki/xacro" name="robot">
     <xacro:include filename="robot_core.xacro" />
-    <xacro:include filename="gz_control.xacro" />
+    <!-- <xacro:include filename="gz_control.xacro" /> -->
+    <xacro:include filename="ros2_control.xacro" />
+    <xacro:include filename="camera.xacro" />
 </robot>

File: ros2_ws/src/lunabot_2425/description/robot_core.xacro (robot description, xacro)
@@ -9,4 +9,7 @@
     <material name="grey">
         <color rgba="0.7 0.7 0.7 1" />
+    </material>
+    <material name="green">
+        <color rgba="0.1 0.8 0.1 1" />
     </material>
     <material name="black">
@@ -43,5 +46,5 @@
     </link>
     <!-- REAR LEFT WHEEL POD ASSEMBLY -->
-    <joint name="rear_left_steer_joint" type="continuous">
+    <joint name="rear_left_steer_joint" type="fixed">
         <parent link="chassis" />
         <child link="rear_left_pod" />
@@ -92,5 +95,5 @@
     </link>
     <!-- REAR RIGHT WHEEL POD ASSEMBLY -->
-    <joint name="rear_right_steer_joint" type="continuous">
+    <joint name="rear_right_steer_joint" type="fixed">
         <parent link="chassis" />
         <child link="rear_right_pod" />
@@ -141,5 +144,5 @@
     </link>
     <!-- FRONT LEFT WHEEL POD ASSEMBLY -->
-    <joint name="front_left_steer_joint" type="continuous">
+    <joint name="front_left_steer_joint" type="fixed">
         <parent link="chassis" />
         <child link="front_left_pod" />
@@ -190,5 +193,5 @@
     </link>
     <!-- FRONT RIGHT WHEEL POD ASSEMBLY -->
-    <joint name="front_right_steer_joint" type="continuous">
+    <joint name="front_right_steer_joint" type="fixed">
         <parent link="chassis" />
         <child link="front_right_pod" />
