Commit message: custom controller functioning, but the kinematics math is very wrong

File: ros2_ws/src/lunabot_2425/description/robot_core.xacro (robot description, xacro)
@@ -46,5 +46,5 @@
     </link>
     <!-- REAR LEFT WHEEL POD ASSEMBLY -->
-    <joint name="rear_left_steer_joint" type="fixed">
+    <joint name="rear_left_steer_joint" type="continuous">
         <parent link="chassis" />
         <child link="rear_left_pod" />
@@ -95,5 +95,5 @@
     </link>
     <!-- REAR RIGHT WHEEL POD ASSEMBLY -->
-    <joint name="rear_right_steer_joint" type="fixed">
+    <joint name="rear_right_steer_joint" type="continuous">
         <parent link="chassis" />
         <child link="rear_right_pod" />
@@ -144,5 +144,5 @@
     </link>
     <!-- FRONT LEFT WHEEL POD ASSEMBLY -->
-    <joint name="front_left_steer_joint" type="fixed">
+    <joint name="front_left_steer_joint" type="continuous">
         <parent link="chassis" />
         <child link="front_left_pod" />
@@ -193,5 +193,5 @@
     </link>
     <!-- FRONT RIGHT WHEEL POD ASSEMBLY -->
-    <joint name="front_right_steer_joint" type="fixed">
+    <joint name="front_right_steer_joint" type="continuous">
         <parent link="chassis" />
         <child link="front_right_pod" />

File: ros2_ws/src/lunabot_2425/description/ros2_control.xacro (robot description, xacro)
@@ -37,4 +37,36 @@
             <state_interface name="position"/>
         </joint>
+        <joint name="rear_left_steer_joint">
+            <command_interface name="position">
+                <param name="min">-95</param>
+                <param name="max">95</param>
+            </command_interface>
+            <state_interface name="velocity"/>
+            <state_interface name="position"/>
+        </joint>
+        <joint name="rear_right_steer_joint">
+            <command_interface name="position">
+                <param name="min">-95</param>
+                <param name="max">95</param>
+            </command_interface>
+            <state_interface name="velocity"/>
+            <state_interface name="position"/>
+        </joint>
+        <joint name="front_left_steer_joint">
+            <command_interface name="position">
+                <param name="min">-95</param>
+                <param name="max">95</param>
+            </command_interface>
+            <state_interface name="velocity"/>
+            <state_interface name="position"/>
+        </joint>
+        <joint name="front_right_steer_joint">
+            <command_interface name="position">
+                <param name="min">-95</param>
+                <param name="max">95</param>
+            </command_interface>
+            <state_interface name="velocity"/>
+            <state_interface name="position"/>
+        </joint>
     </ros2_control>
     <gazebo>
