Commit message: rotate depth camera down

File: ros2_ws/src/lunabot_2425/description/depth_camera.xacro (robot description, xacro)
@@ -4,5 +4,5 @@
         <parent link="base_link" />
         <child link="depth_camera_link" />
-        <origin xyz="0.275 0.25 1.17" rpy="0 0.2 0" />
+        <origin xyz="0.275 0.25 1.17" rpy="0 0.6 0" />
     </joint>
     <link name="depth_camera_link">

Commit message: move depth camera closer to regular camera

File: ros2_ws/src/lunabot_2425/description/depth_camera.xacro (robot description, xacro)
@@ -4,5 +4,5 @@
         <parent link="base_link" />
         <child link="depth_camera_link" />
-        <origin xyz="0.275 0.25 1.17" rpy="0 0.6 0" />
+        <origin xyz="0.275 0.15 1.17" rpy="0 0.6 0" />
     </joint>
     <link name="depth_camera_link">

Commit message: move depth camera to same position as regular camera

File: ros2_ws/src/lunabot_2425/description/depth_camera.xacro (robot description, xacro)
@@ -4,5 +4,5 @@
         <parent link="base_link" />
         <child link="depth_camera_link" />
-        <origin xyz="0.275 0.15 1.17" rpy="0 0.6 0" />
+        <origin xyz="0.275 0.12 1.17" rpy="0 0.6 0" />
     </joint>
     <link name="depth_camera_link">
