Commit message: remove unused tags from camera.xacro

File: ros2_ws/src/lunabot_2425/description/camera.xacro (robot description, xacro)
@@ -15,10 +15,4 @@
         </visual>
     </link>
-    <joint name="camera_optical_joint" type="fixed">
-        <parent link="camera_link" />
-        <child link="camera_link_optical" />
-        <origin xyz="0 0 0" rpy="-1.57079632679489 0 -1.57079632679489" />
-    </joint>
-    <link name="camera_link_optical"></link>
     <gazebo reference="camera_link">
         <sensor name="camera" type="camera">
@@ -39,5 +33,4 @@
             </camera>
             <topic>camera/image_raw</topic>
-            <!-- <gz_frame_id>camera_link_optical</gz_frame_id> -->
         </sensor>
     </gazebo>

Commit message: rotate camera down to match depth camera

File: ros2_ws/src/lunabot_2425/description/camera.xacro (robot description, xacro)
@@ -4,5 +4,5 @@
         <parent link="base_link" />
         <child link="camera_link" />
-        <origin xyz="0.275 0.12 1.17" rpy="0 0.2 0" />
+        <origin xyz="0.275 0.12 1.17" rpy="0 0.6 0" />
     </joint>
     <link name="camera_link">

Commit message: add optical link for rgb camera

File: ros2_ws/src/lunabot_2425/description/camera.xacro (robot description, xacro)
@@ -15,4 +15,10 @@
         </visual>
     </link>
+    <joint name="camera_optical_joint" type="fixed">
+        <parent link="camera_link" />
+        <child link="camera_link_optical" />
+        <origin xyz="0 0 0" rpy="-1.57079632679 0 -1.57079632679" />
+    </joint>
+    <link name="camera_link_optical"></link>
     <gazebo reference="camera_link">
         <sensor name="camera" type="camera">
@@ -33,5 +39,5 @@
             <update_rate>15</update_rate>
             <topic>camera/image_raw</topic>
-            <gz_frame_id>camera_link</gz_frame_id>
+            <gz_frame_id>camera_link_optical</gz_frame_id>
         </sensor>
     </gazebo>
